File: hardware/edid-injector.kicad_pcb (KiCad board)
At the start: 2 copper layers, 42 parts, among them SW1 SW_PUSH, U1 C8051F381/3/5/7/C-GQ

Commit message: Connect everything up.
Parts:
- RRST1: moved to F.Cu
- moved DUSB1 40.5 mm to (126.1, 99.4)
- moved JEDID1 29.8 mm to (113.1, 79.2), turned to 0 degrees
- moved SW1 29.6 mm to (131.1, 92.6), turned to 90 degrees
- moved RUSB1 28.0 mm to (125.6, 94.6)
- moved LUSB1 26.0 mm to (126.2, 92.3), turned to 0 degrees
- moved JCEC1 24.7 mm to (106.2, 79.1)
- moved L7 11.9 mm to (110.4, 113.0)
- moved RL7 9.93 mm to (112.9, 111.7), turned to 180 degrees
- moved CDBG1 9.38 mm to (121.2, 91.4), turned to 0 degrees
- moved RL14 9.10 mm to (110.6, 105.1)
- moved L16 9.00 mm to (107.8, 100.0)
- moved L14 8.96 mm to (107.8, 105.1)
- moved L15 8.91 mm to (107.8, 102.5)
- moved L17 8.91 mm to (107.8, 97.4)
- moved RL17 8.90 mm to (111.5, 97.7)
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Routing:
- net GND: track 0.00 -> 178.7 mm, vias 0 -> 11
- net /SRC_HPD: track 0.00 -> 79.2 mm, vias 0 -> 6
- net /SRC_CEC: track 0.00 -> 76.0 mm, vias 0 -> 3
- net /VHDMI: track 0.00 -> 73.9 mm, vias 0 -> 2
- net /SRC_SCL: track 0.00 -> 54.6 mm, vias 0 -> 5
- net /VCC5V0: track 0.00 -> 52.2 mm, vias 0 -> 3
- net /SRC_SDA: track 0.00 -> 51.8 mm, vias 0 -> 3
- net /SINK_CEC: track 0.00 -> 45.6 mm, vias 0 -> 4
- net /SINK_SCL: track 0.00 -> 45.2 mm, vias 0 -> 2
- net /SINK_SDA: track 0.00 -> 44.2 mm, vias 0 -> 2
- net /SINK_HPD: track 0.00 -> 42.9 mm, vias 0 -> 2
- net Net-(RSEGC1-Pad1): track 0.00 -> 42.8 mm, vias 0 -> 4
- net Net-(RSEGP1-Pad1): track 0.00 -> 32.7 mm, vias 0 -> 4
- net Net-(RSEGA1-Pad1): track 0.00 -> 27.1 mm, vias 0 -> 2
- net Net-(RSEGE1-Pad1): track 0.00 -> 26.2 mm, vias 0 -> 2
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
Commit message: Old changes.
Routing:
- net /SRC_CEC: track 76.0 -> 76.7 mm
- added copper zone on F.Cu, net GND
