File: hardware/hdmi/edid-injector.sch (KiCad schematic (older format))
At the start: 42 parts, among them SW1 SW_PUSH, U1 C8051F381/3/5/7/C-GQ

Commit message: Bunch of small tweaks.
Parts:
- removed CDBG1, JCEC1: CONN_01X02, Pin_Headers:Pin_Header_Straight_1x02, symbol CONN_01X02
- removed JEDID1: CONN_02X03, Pin_Headers:Pin_Header_Straight_2x03, symbol CONN_02X03
- added CDBG1: CONN_01X04, symbol CONN_01X04
- added JCEC1: CONN_01X05, symbol CONN_01X05
- added JEDID1: CONN_02X05, symbol CONN_02X05
- added LPWR2: LED, LEDs:LED-0805, symbol LED-RESCUE-edid-injector
- added RPWR2: R, Resistors_SMD:R_0402, symbol R-RESCUE-edid-injector
- L14, L15, L16, L17, L4, L5, L6, L7, LHDMI1, LPWR1, LUSB1: symbol LED -> LED-RESCUE-edid-injector
- RHDMI1, RL14, RL15, RL16, RL17, RL4, RL5, RL6, RL7, RPWR1, RRST1, RSEGA1, RSEGB1, RSEGC1, RSEGD1, RSEGE1, RSEGF1, RSEGG1, RSEGP1, RUSB1: symbol R -> R-RESCUE-edid-injector
Connections:
- net GND: now also CDBG1.1 (P1), JCEC1.5 (P5), JEDID1.7 (P7), JEDID1.8 (P8), LPWR2.2 (K)
- net SINK_CEC: now also JCEC1.3 (P3)
- net SINK_HPD: now also JEDID1.6 (P6)
- net SINK_SCL: now also JEDID1.2 (P2)
- net SINK_SDA: now also JEDID1.4 (P4)
- net SRC_CEC: now also JCEC1.2 (P2)
- net SRC_HPD: now also JEDID1.1 (P1)
- net SRC_SCL: now also JEDID1.5 (P5)
- net SRC_SDA: now also JEDID1.3 (P3)
- net VCC3V3: now also CDBG1.4 (P4), JCEC1.4 (P4), JEDID1.10 (P10), JEDID1.9 (P9), RPWR2.2
- net RES: now reaches CSINK1.14 (RES)
- net RES: now also CSRC1.14 (RES)
- net at U1.10 (P3.0/C2D): now also CDBG1.3 (P3)
- net at RRST1.1, SW1.1, U1.9 (~RST~/C2CK): now also CDBG1.2 (P2)
- new net: LPWR2.1 (A), RPWR2.1
- no-connect marks 3 -> 2

Commit message: Fixing component assignments.
Parts:
- CDBG1: footprint (none) -> Pin_Headers:Pin_Header_Straight_1x04
- JCEC1: footprint (none) -> Pin_Headers:Pin_Header_Straight_1x05
- JEDID1: footprint (none) -> Pin_Headers:Pin_Header_Straight_2x05
- LPWR2: footprint LEDs:LED-0805 -> LEDs:LED_0805
Changed lines of the file:
@@
 F 0 "JEDID1" H 5225 4050 50  0000 C CNN
 F 1 "CONN_02X05" H 5225 3450 50  0000 C CNN
-F 2 "" H 5225 2550 50  0000 C CNN
+F 2 "Pin_Headers:Pin_Header_Straight_2x05" H 5225 2550 50  0001 C CNN
 F 3 "" H 5225 2550 50  0000 C CNN
 	1    5225 3750
@@
 F 0 "JCEC1" H 4500 2700 50  0000 C CNN
 F 1 "CONN_01X05" V 4550 3000 50  0000 C CNN
-F 2 "" H 4450 3000 50  0000 C CNN
+F 2 "Pin_Headers:Pin_Header_Straight_1x05" H 4450 3000 50  0001 C CNN
 F 3 "" H 4450 3000 50  0000 C CNN
 	1    4450 3000
@@
 F 0 "LPWR2" H 6850 4700 50  0000 C CNN
 F 1 "LED" H 6850 4500 50  0000 C CNN
-F 2 "LEDs:LED-0805" H 6850 4600 60  0001 C CNN
+F 2 "LEDs:LED_0805" H 6850 4600 60  0001 C CNN
 F 3 "" H 6850 4600 60  0000 C CNN
 	1    6850 4600
@@
 F 0 "CDBG1" H 5450 6000 50  0000 C CNN
 F 1 "CONN_01X04" V 5550 5750 50  0000 C CNN
-F 2 "" H 5450 5750 50  0000 C CNN
+F 2 "Pin_Headers:Pin_Header_Straight_1x04" H 5450 5750 50  0001 C CNN
 F 3 "" H 5450 5750 50  0000 C CNN
 	1    5450 5750

Commit message: Trying to make things a little more uniform.
Parts:
- L14, L15, L16, L17, L4, L5, L6, L7, LHDMI1, LPWR1, LUSB1: footprint LEDs:LED-0805 -> LEDs:LED_0805
Changed lines of the file:
@@
 F 0 "LPWR1" H 3750 4500 50  0000 C CNN
 F 1 "LED" H 3750 4300 50  0000 C CNN
-F 2 "LEDs:LED-0805" H 3750 4400 60  0001 C CNN
+F 2 "LEDs:LED_0805" H 3750 4400 60  0001 C CNN
 F 3 "" H 3750 4400 60  0000 C CNN
 	1    3750 4400
@@
 F 0 "LHDMI1" H 1350 3200 50  0000 C CNN
 F 1 "LED" H 1350 3000 50  0000 C CNN
-F 2 "LEDs:LED-0805" H 1350 3100 60  0001 C CNN
+F 2 "LEDs:LED_0805" H 1350 3100 60  0001 C CNN
 F 3 "" H 1350 3100 60  0000 C CNN
 	1    1350 3100
@@
 F 0 "LUSB1" H 1350 3500 50  0000 C CNN
 F 1 "LED" H 1350 3300 50  0000 C CNN
-F 2 "LEDs:LED-0805" H 1350 3400 60  0001 C CNN
+F 2 "LEDs:LED_0805" H 1350 3400 60  0001 C CNN
 F 3 "" H 1350 3400 60  0000 C CNN
 	1    1350 3400
@@
 F 0 "L4" H 8950 3350 50  0000 C CNN
 F 1 "LED" H 9350 3350 50  0000 C CNN
-F 2 "LEDs:LED-0805" H 9150 3300 60  0001 C CNN
+F 2 "LEDs:LED_0805" H 9150 3300 60  0001 C CNN
 F 3 "" H 9150 3300 60  0000 C CNN
 	1    9150 3300
@@
 F 0 "L5" H 8450 3450 50  0000 C CNN
 F 1 "LED" H 8850 3450 50  0000 C CNN
-F 2 "LEDs:LED-0805" H 8650 3400 60  0001 C CNN
+F 2 "LEDs:LED_0805" H 8650 3400 60  0001 C CNN
 F 3 "" H 8650 3400 60  0000 C CNN
 	1    8650 3400
@@
 F 0 "L6" H 8950 3550 50  0000 C CNN
 F 1 "LED" H 9350 3550 50  0000 C CNN
-F 2 "LEDs:LED-0805" H 9150 3500 60  0001 C CNN
+F 2 "LEDs:LED_0805" H 9150 3500 60  0001 C CNN
 F 3 "" H 9150 3500 60  0000 C CNN
 	1    9150 3500
@@
 F 0 "L7" H 8450 3650 50  0000 C CNN
 F 1 "LED" H 8850 3650 50  0000 C CNN
-F 2 "LEDs:LED-0805" H 8650 3600 60  0001 C CNN
+F 2 "LEDs:LED_0805" H 8650 3600 60  0001 C CNN
 F 3 "" H 8650 3600 60  0000 C CNN
 	1    8650 3600
@@
 F 0 "L14" H 8950 4450 50  0000 C CNN
 F 1 "LED" H 9350 4450 50  0000 C CNN
-F 2 "LEDs:LED-0805" H 9150 4400 60  0001 C CNN
+F 2 "LEDs:LED_0805" H 9150 4400 60  0001 C CNN
 F 3 "" H 9150 4400 60  0000 C CNN
 	1    9150 4400
@@
 F 0 "L15" H 8450 4550 50  0000 C CNN
 F 1 "LED" H 8850 4550 50  0000 C CNN
-F 2 "LEDs:LED-0805" H 8650 4500 60  0001 C CNN
+F 2 "LEDs:LED_0805" H 8650 4500 60  0001 C CNN
 F 3 "" H 8650 4500 60  0000 C CNN
 	1    8650 4500
@@
 F 0 "L16" H 8950 4650 50  0000 C CNN
 F 1 "LED" H 9350 4650 50  0000 C CNN
-F 2 "LEDs:LED-0805" H 9150 4600 60  0001 C CNN
+F 2 "LEDs:LED_0805" H 9150 4600 60  0001 C CNN
 F 3 "" H 9150 4600 60  0000 C CNN
 	1    9150 4600
@@
 F 0 "L17" H 8450 4750 50  0000 C CNN
 F 1 "LED" H 8850 4750 50  0000 C CNN
-F 2 "LEDs:LED-0805" H 8650 4700 60  0001 C CNN
+F 2 "LEDs:LED_0805" H 8650 4700 60  0001 C CNN
 F 3 "" H 8650 4700 60  0000 C CNN
 	1    8650 4700

Commit message: Tweaking.
Connections:
- net GND: now also JCEC1.4 (P4); no longer JCEC1.5 (P5)
- net VCC3V3: now also JCEC1.5 (P5); no longer JCEC1.4 (P4)
Changed lines of the file:
@@
 	5125 3375 4750 3375
 Wire Wire Line
-	4750 3200 4750 4125
+	4750 3100 4750 4125
 Wire Wire Line
 	4750 4125 5125 4125
@@
 	4825 4050 5025 4050
 Wire Wire Line
-	4825 3100 4825 4050
+	4825 3200 4825 4050
 Connection ~ 5025 4050
 Wire Wire Line
@@
 	-1   0    0    -1
 $EndComp
-Wire Wire Line
-	4750 3200 4650 3200
 Connection ~ 4750 3375
-Wire Wire Line
-	4825 3100 4650 3100
 Connection ~ 4825 3450
 NoConn ~ 4650 2800
@@
 Wire Wire Line
 	6700 5700 6700 5900
+Wire Wire Line
+	4750 3100 4650 3100
+Wire Wire Line
+	4825 3200 4650 3200
 $EndSCHEMATC
